File: PCAL6534EV-breakout.kicad_sch (KiCad schematic)
At the start: 14 parts, among them J1 SM04B-SRSS-TB, J2 Conn_01x20, J3 Conn_01x20, J4 Conn_02x04_Odd_Even, U1 PCAL6534EV

Commit message: add more art
Parts:
- JP2, JP3, JP4: now left out of the parts list
Changed lines of the file:
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@@
 		(unit 1)
 		(exclude_from_sim no)
-		(in_bom yes)
+		(in_bom no)
 		(on_board yes)
 		(dnp no)
@@
 		(unit 1)
 		(exclude_from_sim no)
-		(in_bom yes)
+		(in_bom no)
 		(on_board yes)
 		(dnp no)
@@
 		(unit 1)
 		(exclude_from_sim no)
-		(in_bom yes)
-		(on_board yes)
-		(dnp no)
+		(in_bom no)
+		(on_board yes)
+		(dnp no)
